File: neptune/data_management.kicad_sch (KiCad schematic)
At the start: 5 parts, among them J1 Conn_Coaxial, J7 THD2528-11SD-GF, U5 RFM95W-915S2

Commit message: Updated some footprints, restarted routing
Parts:
- J1: footprint Connector_Coaxial:SMA_Amphenol_132291_Vertical -> Connector_Coaxial:U.FL_Molex_MCRF_73412-0110_Vertical
Changed lines of the file:
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@@
       (effects (font (size 1.27 1.27)) (justify left))
     )
-    (property "Footprint" "Connector_Coaxial:SMA_Amphenol_132291_Vertical" (at 66.04 64.77 0)
+    (property "Footprint" "Connector_Coaxial:U.FL_Molex_MCRF_73412-0110_Vertical" (at 66.04 64.77 0)
       (effects (font (size 1.27 1.27)) hide)
     )

Commit message: Continued routing
Parts:
- removed J7: THD2528-11SD-GF, local-library:THD252811SDGF, symbol THD2528-11SD-GF:THD2528-11SD-GF
- added U10: AT25SF081-XMHF-X, Package_SO:SOP-8_5.28x5.23mm_P1.27mm, symbol Memory_Flash:AT25SF081-XMHF-X
Connections:
- net +3.3V: now also U10.8 (VCC)
- net GND: now also U10.4 (GND)
- new net CS_FC: U10.1 (~{CS})
- new net HOLD_FC: U10.7 (~{HOLD}/IO3)
- new net MISO_FC: U10.2 (SO/IO1)
- new net MOSI_FC: U10.5 (SI/IO0)
- new net SCK_FC: U10.6 (SCK)
- new net WP_FC: U10.3 (~{WP}/IO2)
- no-connect marks 7 -> 5
Other:
- note added: "Flash chip"
- note removed: "SD card"

Commit message: Routed 3.3V stepdown, added indicator LEDs
Connections:
- net +3.3V renamed +3V3
Changed lines of the file:
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@@
     (stroke (width 0) (type default))
   )
-  (wire (pts (xy 73.66 45.72) (xy 67.31 45.72))
+  (wire (pts (xy 67.31 45.72) (xy 73.66 45.72))
     (stroke (width 0) (type default))
   )
@@
     (stroke (width 0) (type default))
   )
+  (wire (pts (xy 34.29 77.47) (xy 31.75 77.47))
+    (stroke (width 0) (type default))
+  )
+  (wire (pts (xy 67.31 53.34) (xy 73.66 53.34))
+    (stroke (width 0) (type default))
+  )
+  (wire (pts (xy 31.75 64.77) (xy 34.29 64.77))
+    (stroke (width 0) (type default))
+  )
+  (wire (pts (xy 31.75 67.31) (xy 34.29 67.31))
+    (stroke (width 0) (type default))
+  )
+  (polyline (pts (xy 100.33 38.1) (xy 100.33 81.28))
+    (stroke (width 0) (type default))
+  )
+  (wire (pts (xy 49.53 87.63) (xy 49.53 91.44))
+    (stroke (width 0) (type default))
+  )
+  (wire (pts (xy 73.66 53.34) (xy 80.01 53.34))
+    (stroke (width 0) (type default))
+  )
+  (polyline (pts (xy 19.05 97.79) (xy 90.17 97.79))
+    (stroke (width 0) (type default))
+  )
+  (wire (pts (xy 46.99 87.63) (xy 46.99 91.44))
+    (stroke (width 0) (type default))
+  )
+  (polyline (pts (xy 90.17 97.79) (xy 90.17 38.1))
+    (stroke (width 0) (type default))
+  )
+  (wire (pts (xy 114.3 57.15) (xy 116.84 57.15))
+    (stroke (width 0) (type default))
+  )
+  (wire (pts (xy 114.3 64.77) (xy 116.84 64.77))
+    (stroke (width 0) (type default))
+  )
+  (wire (pts (xy 44.45 91.44) (xy 46.99 91.44))
+    (stroke (width 0) (type default))
+  )
+  (wire (pts (xy 114.3 59.69) (xy 116.84 59.69))
+    (stroke (width 0) (type default))
+  )
+  (wire (pts (xy 114.3 52.07) (xy 116.84 52.07))
+    (stroke (width 0) (type default))
+  )
   (wire (pts (xy 73.66 45.72) (xy 80.01 45.72))
-    (stroke (width 0) (type default))
-  )
-  (wire (pts (xy 34.29 77.47) (xy 31.75 77.47))
-    (stroke (width 0) (type default))
-  )
-  (wire (pts (xy 67.31 53.34) (xy 73.66 53.34))
-    (stroke (width 0) (type default))
-  )
-  (wire (pts (xy 31.75 64.77) (xy 34.29 64.77))
-    (stroke (width 0) (type default))
-  )
-  (wire (pts (xy 31.75 67.31) (xy 34.29 67.31))
-    (stroke (width 0) (type default))
-  )
-  (polyline (pts (xy 100.33 38.1) (xy 100.33 81.28))
-    (stroke (width 0) (type default))
-  )
-  (wire (pts (xy 49.53 87.63) (xy 49.53 91.44))
-    (stroke (width 0) (type default))
-  )
-  (wire (pts (xy 73.66 53.34) (xy 80.01 53.34))
-    (stroke (width 0) (type default))
-  )
-  (polyline (pts (xy 19.05 97.79) (xy 90.17 97.79))
-    (stroke (width 0) (type default))
-  )
-  (wire (pts (xy 46.99 87.63) (xy 46.99 91.44))
-    (stroke (width 0) (type default))
-  )
-  (polyline (pts (xy 90.17 97.79) (xy 90.17 38.1))
-    (stroke (width 0) (type default))
-  )
-  (wire (pts (xy 114.3 57.15) (xy 116.84 57.15))
-    (stroke (width 0) (type default))
-  )
-  (wire (pts (xy 114.3 64.77) (xy 116.84 64.77))
-    (stroke (width 0) (type default))
-  )
-  (wire (pts (xy 44.45 91.44) (xy 46.99 91.44))
-    (stroke (width 0) (type default))
-  )
-  (wire (pts (xy 114.3 59.69) (xy 116.84 59.69))
-    (stroke (width 0) (type default))
-  )
-  (wire (pts (xy 114.3 52.07) (xy 116.84 52.07))
     (stroke (width 0) (type default))
   )
@@
     (effects (font (size 1.27 1.27)) (justify left))
   )
-  (symbol (lib_id "power:+3.3V") (at 46.99 57.15 0) (unit 1)
-    (in_bom yes) (on_board yes) (dnp no) (fields_autoplaced)
-    (property "Reference" "#PWR06" (at 46.99 60.96 0)
-      (effects (font (size 1.27 1.27)) hide)
-    )
-    (property "Value" "+3.3V" (at 46.99 53.34 0)
-      (effects (font (size 1.27 1.27)))
-    )
-    (property "Footprint" "" (at 46.99 57.15 0)
-      (effects (font (size 1.27 1.27)) hide)
-    )
-    (property "Datasheet" "" (at 46.99 57.15 0)
-      (effects (font (size 1.27 1.27)) hide)
-    )
-    (pin "1")
-    (instances
-      (project "neptune"
-        (path "/e63e39d7-6ac0-4ffd-8aa3-1841a4541b55/b694d9b6-8e2a-4217-a81b-e156ec88b46a"
-          (reference "#PWR06") (unit 1)
-        )
-      )
-    )
-  )
   (symbol (lib_id "Device:C_Small") (at 80.01 49.53 0) (unit 1)
     (in_bom yes) (on_board yes) (dnp no)
@@
     )
   )
+  (symbol (lib_id "power:+3V3") (at 127 46.99 0) (unit 1)
+    (in_bom yes) (on_board yes) (dnp no) (fields_autoplaced)
+    (property "Reference" "#PWR04" (at 127 50.8 0)
+      (effects (font (size 1.27 1.27)) hide)
+    )
+    (property "Value" "+3V3" (at 127 43.18 0)
+      (effects (font (size 1.27 1.27)))
+    )
+    (property "Footprint" "" (at 127 46.99 0)
+      (effects (font (size 1.27 1.27)) hide)
+    )
+    (property "Datasheet" "" (at 127 46.99 0)
+      (effects (font (size 1.27 1.27)) hide)
+    )
+    (pin "1")
+    (instances
+      (project "neptune"
+        (path "/e63e39d7-6ac0-4ffd-8aa3-1841a4541b55/761c8e29-382a-475c-a37a-7201cc9cd0f5"
+          (reference "#PWR04") (unit 1)
+        )
+        (path "/e63e39d7-6ac0-4ffd-8aa3-1841a4541b55/b694d9b6-8e2a-4217-a81b-e156ec88b46a"
+          (reference "#PWR039") (unit 1)
+        )
+      )
+    )
+  )
   (symbol (lib_id "power:GND") (at 46.99 91.44 0) (unit 1)
     (in_bom yes) (on_board yes) (dnp no)
@@
         (path "/e63e39d7-6ac0-4ffd-8aa3-1841a4541b55/b694d9b6-8e2a-4217-a81b-e156ec88b46a"
           (reference "#PWR037") (unit 1)
-        )
-      )
-    )
-  )
-  (symbol (lib_id "power:+3.3V") (at 127 46.99 0) (unit 1)
-    (in_bom yes) (on_board yes) (dnp no) (fields_autoplaced)
-    (property "Reference" "#PWR039" (at 127 50.8 0)
-      (effects (font (size 1.27 1.27)) hide)
-    )
-    (property "Value" "+3.3V" (at 127 43.18 0)
-      (effects (font (size 1.27 1.27)))
-    )
-    (property "Footprint" "" (at 127 46.99 0)
-      (effects (font (size 1.27 1.27)) hide)
-    )
-    (property "Datasheet" "" (at 127 46.99 0)
-      (effects (font (size 1.27 1.27)) hide)
-    )
-    (pin "1")
-    (instances
-      (project "neptune"
-        (path "/e63e39d7-6ac0-4ffd-8aa3-1841a4541b55/b694d9b6-8e2a-4217-a81b-e156ec88b46a"
-          (reference "#PWR039") (unit 1)
         )
       )
@@
         (path "/e63e39d7-6ac0-4ffd-8aa3-1841a4541b55/b694d9b6-8e2a-4217-a81b-e156ec88b46a"
           (reference "#PWR040") (unit 1)
+        )
+      )
+    )
+  )
+  (symbol (lib_id "power:+3V3") (at 46.99 57.15 0) (unit 1)
+    (in_bom yes) (on_board yes) (dnp no) (fields_autoplaced)
+    (property "Reference" "#PWR04" (at 46.99 60.96 0)
+      (effects (font (size 1.27 1.27)) hide)
+    )
+    (property "Value" "+3V3" (at 46.99 53.34 0)
+      (effects (font (size 1.27 1.27)))
+    )
+    (property "Footprint" "" (at 46.99 57.15 0)
+      (effects (font (size 1.27 1.27)) hide)
+    )
+    (property "Datasheet" "" (at 46.99 57.15 0)
+      (effects (font (size 1.27 1.27)) hide)
+    )
+    (pin "1")
+    (instances
+      (project "neptune"
+        (path "/e63e39d7-6ac0-4ffd-8aa3-1841a4541b55/761c8e29-382a-475c-a37a-7201cc9cd0f5"
+          (reference "#PWR04") (unit 1)
+        )
+        (path "/e63e39d7-6ac0-4ffd-8aa3-1841a4541b55/b694d9b6-8e2a-4217-a81b-e156ec88b46a"
+          (reference "#PWR06") (unit 1)
         )
       )
@@
     )
   )
-  (symbol (lib_id "power:+3.3V") (at 73.66 45.72 0) (unit 1)
+  (symbol (lib_id "power:+3V3") (at 73.66 45.72 0) (unit 1)
     (in_bom yes) (on_board yes) (dnp no) (fields_autoplaced)
-    (property "Reference" "#PWR?" (at 73.66 49.53 0)
-      (effects (font (size 1.27 1.27)) hide)
-    )
-    (property "Value" "+3.3V" (at 73.66 40.64 0)
+    (property "Reference" "#PWR04" (at 73.66 49.53 0)
+      (effects (font (size 1.27 1.27)) hide)
+    )
+    (property "Value" "+3V3" (at 73.66 41.91 0)
       (effects (font (size 1.27 1.27)))
     )
@@
     (instances
       (project "neptune"
-        (path "/e63e39d7-6ac0-4ffd-8aa3-1841a4541b55/fd0daead-056b-49b0-b136-e76d44737a4c"
-          (reference "#PWR?") (unit 1)
-        )
-        (path "/e63e39d7-6ac0-4ffd-8aa3-1841a4541b55/b694d9b6-8e2a-4217-a81b-e156ec88b46a"
+        (path "/e63e39d7-6ac0-4ffd-8aa3-1841a4541b55/761c8e29-382a-475c-a37a-7201cc9cd0f5"
+          (reference "#PWR04") (unit 1)
+        )
+        (path "/e63e39d7-6ac0-4ffd-8aa3-1841a4541b55/b694d9b6-8e2a-4217-a81b-e156ec88b46a"
