File: neptune/neptune.kicad_sch (KiCad schematic)
At the start: 8 parts

Commit message: Updated some footprints, restarted routing
Parts:
- TP1, TP2, TP3, TP4: footprint TestPoint:TestPoint_Pad_D2.0mm -> TestPoint:TestPoint_Pad_D1.0mm
Changed lines of the file:
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@@
       (effects (font (size 1.27 1.27)) (justify right))
     )
-    (property "Footprint" "TestPoint:TestPoint_Pad_D2.0mm" (at 27.94 146.05 0)
+    (property "Footprint" "TestPoint:TestPoint_Pad_D1.0mm" (at 27.94 146.05 0)
       (effects (font (size 1.27 1.27)) hide)
     )
@@
       (effects (font (size 1.27 1.27)) (justify right))
     )
-    (property "Footprint" "TestPoint:TestPoint_Pad_D2.0mm" (at 45.72 146.05 0)
+    (property "Footprint" "TestPoint:TestPoint_Pad_D1.0mm" (at 45.72 146.05 0)
       (effects (font (size 1.27 1.27)) hide)
     )
@@
       (effects (font (size 1.27 1.27)) (justify left))
     )
-    (property "Footprint" "TestPoint:TestPoint_Pad_D2.0mm" (at 46.99 156.21 0)
+    (property "Footprint" "TestPoint:TestPoint_Pad_D1.0mm" (at 46.99 156.21 0)
       (effects (font (size 1.27 1.27)) hide)
     )
@@
       (effects (font (size 1.27 1.27)) (justify right))
     )
-    (property "Footprint" "TestPoint:TestPoint_Pad_D2.0mm" (at 36.83 146.05 0)
+    (property "Footprint" "TestPoint:TestPoint_Pad_D1.0mm" (at 36.83 146.05 0)
       (effects (font (size 1.27 1.27)) hide)
     )

Commit message: Continued routing
Other:
- sheet Data management ports: added CS_FC, HOLD_FC, MISO_FC, MOSI_FC, SCK_FC, WP_FC; removed CLK_SD, CS_SD, MISO_SD, MOSI_SD
- sheet STM32 ports: added CS_FC, HOLD_FC, MISO_FC, MOSI_FC, SCK_FC, WP_FC; removed CLK_SD, CS_SD, MISO_SD, MOSI_SD
Changed lines of the file:
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@@
+    (stroke (width 0) (type default))
+  )
+  (wire (pts (xy 171.45 46.99) (xy 165.1 46.99))
+    (stroke (width 0) (type default))
+  )
+  (wire (pts (xy 165.1 77.47) (xy 177.8 77.47))
+    (stroke (width 0) (type default))
+  )
+  (wire (pts (xy 101.6 120.65) (xy 114.3 120.65))
+    (stroke (width 0) (type default))
+  )
+  (wire (pts (xy 101.6 99.06) (xy 114.3 99.06))
+    (stroke (width 0) (type default))
+  )
+  (wire (pts (xy 101.6 113.03) (xy 114.3 113.03))
+    (stroke (width 0) (type default))
+  )
+  (wire (pts (xy 101.6 101.6) (xy 114.3 101.6))
+    (stroke (width 0) (type default))
+  )
+  (wire (pts (xy 101.6 104.14) (xy 114.3 104.14))
+    (stroke (width 0) (type default))
+  )
+  (wire (pts (xy 177.8 71.12) (xy 171.45 71.12))
+    (stroke (width 0) (type default))
+  )
+  (wire (pts (xy 165.1 74.93) (xy 177.8 74.93))
+    (stroke (width 0) (type default))
+  )
+  (wire (pts (xy 165.1 81.28) (xy 177.8 81.28))
+    (stroke (width 0) (type default))
+  )
+  (wire (pts (xy 165.1 93.98) (xy 177.8 93.98))
+    (stroke (width 0) (type default))
+  )
+  (wire (pts (xy 165.1 87.63) (xy 177.8 87.63))
+    (stroke (width 0) (type default))
+  )
+  (wire (pts (xy 101.6 93.98) (xy 114.3 93.98))
+    (stroke (width 0) (type default))
+  )
+  (wire (pts (xy 165.1 96.52) (xy 177.8 96.52))
+    (stroke (width 0) (type default))
+  )
+  (wire (pts (xy 101.6 96.52) (xy 114.3 96.52))
+    (stroke (width 0) (type default))
+  )
+  (wire (pts (xy 165.1 125.73) (xy 177.8 125.73))
+    (stroke (width 0) (type default))
+  )
+  (wire (pts (xy 165.1 123.19) (xy 177.8 123.19))
+    (stroke (width 0) (type default))
+  )
+  (wire (pts (xy 101.6 115.57) (xy 114.3 115.57))
+    (stroke (width 0) (type default))
+  )
+  (wire (pts (xy 101.6 118.11) (xy 114.3 118.11))
     (stroke (width 0) (type default))
   )
@@
     (stroke (width 0) (type default))
   )
-  (wire (pts (xy 171.45 46.99) (xy 165.1 46.99))
-    (stroke (width 0) (type default))
-  )
-  (wire (pts (xy 165.1 77.47) (xy 177.8 77.47))
-    (stroke (width 0) (type default))
-  )
-  (wire (pts (xy 101.6 99.06) (xy 114.3 99.06))
-    (stroke (width 0) (type default))
-  )
-  (wire (pts (xy 101.6 101.6) (xy 114.3 101.6))
-    (stroke (width 0) (type default))
-  )
-  (wire (pts (xy 101.6 104.14) (xy 114.3 104.14))
-    (stroke (width 0) (type default))
-  )
-  (wire (pts (xy 177.8 71.12) (xy 171.45 71.12))
-    (stroke (width 0) (type default))
-  )
-  (wire (pts (xy 165.1 74.93) (xy 177.8 74.93))
-    (stroke (width 0) (type default))
-  )
-  (wire (pts (xy 165.1 81.28) (xy 177.8 81.28))
-    (stroke (width 0) (type default))
-  )
-  (wire (pts (xy 165.1 93.98) (xy 177.8 93.98))
-    (stroke (width 0) (type default))
-  )
   (wire (pts (xy 101.6 107.95) (xy 114.3 107.95))
-    (stroke (width 0) (type default))
-  )
-  (wire (pts (xy 165.1 87.63) (xy 177.8 87.63))
-    (stroke (width 0) (type default))
-  )
-  (wire (pts (xy 101.6 93.98) (xy 114.3 93.98))
-    (stroke (width 0) (type default))
-  )
-  (wire (pts (xy 165.1 96.52) (xy 177.8 96.52))
-    (stroke (width 0) (type default))
-  )
-  (wire (pts (xy 101.6 96.52) (xy 114.3 96.52))
-    (stroke (width 0) (type default))
-  )
-  (wire (pts (xy 165.1 125.73) (xy 177.8 125.73))
-    (stroke (width 0) (type default))
-  )
-  (wire (pts (xy 165.1 123.19) (xy 177.8 123.19))
-    (stroke (width 0) (type default))
-  )
-  (wire (pts (xy 101.6 115.57) (xy 114.3 115.57))
-    (stroke (width 0) (type default))
-  )
-  (wire (pts (xy 101.6 113.03) (xy 114.3 113.03))
     (stroke (width 0) (type default))
   )
@@
       (effects (font (size 1.27 1.27)) (justify right))
     )
-    (pin "CLK_SD" output (at 114.3 110.49 180)
-      (effects (font (size 1.27 1.27)) (justify left))
-    )
-    (pin "MISO_SD" input (at 114.3 115.57 180)
-      (effects (font (size 1.27 1.27)) (justify left))
-    )
-    (pin "MOSI_SD" output (at 114.3 113.03 180)
-      (effects (font (size 1.27 1.27)) (justify left))
-    )
     (pin "SCK_RF" input (at 114.3 93.98 180)
       (effects (font (size 1.27 1.27)) (justify left))
@@
       (effects (font (size 1.27 1.27)) (justify left))
     )
-    (pin "CS_SD" output (at 114.3 107.95 180)
-      (effects (font (size 1.27 1.27)) (justify left))
-    )
     (pin "RF_100" input (at 114.3 104.14 180)
       (effects (font (size 1.27 1.27)) (justify left))
@@
     (pin "SWDIO" bidirectional (at 165.1 90.17 0)
       (effects (font (size 1.27 1.27)) (justify right))
+    )
+    (pin "MISO_FC" input (at 114.3 113.03 180)
+      (effects (font (size 1.27 1.27)) (justify left))
+    )
+    (pin "SCK_FC" output (at 114.3 115.57 180)
+      (effects (font (size 1.27 1.27)) (justify left))
+    )
+    (pin "MOSI_FC" output (at 114.3 110.49 180)
+      (effects (font (size 1.27 1.27)) (justify left))
+    )
+    (pin "HOLD_FC" output (at 114.3 120.65 180)
+      (effects (font (size 1.27 1.27)) (justify left))
+    )
+    (pin "CS_FC" output (at 114.3 107.95 180)
+      (effects (font (size 1.27 1.27)) (justify left))
+    )
+    (pin "WP_FC" output (at 114.3 118.11 180)
+      (effects (font (size 1.27 1.27)) (justify left))
     )
     (instances
@@
     )
   )
-  (sheet (at 71.12 88.9) (size 30.48 34.29) (fields_autoplaced)
+  (sheet (at 71.12 88.9) (size 30.48 36.83) (fields_autoplaced)
     (stroke (width 0.1524) (type solid))
     (fill (color 0 0 0 0.0000))
@@
       (effects (font (size 1.27 1.27)) (justify left bottom))
     )
-    (property "Sheetfile" "data_management.kicad_sch" (at 71.12 123.7746 0)
+    (property "Sheetfile" "data_management.kicad_sch" (at 71.12 126.3146 0)
       (effects (font (size 1.27 1.27)) (justify left top))
     )
@@
       (effects (font (size 1.27 1.27)) (justify right))
     )
-    (pin "MISO_SD" output (at 101.6 115.57 0)
-      (effects (font (size 1.27 1.27)) (justify right))
-    )
-    (pin "MOSI_SD" input (at 101.6 113.03 0)
-      (effects (font (size 1.27 1.27)) (justify right))
-    )
-    (pin "CLK_SD" input (at 101.6 110.49 0)
-      (effects (font (size 1.27 1.27)) (justify right))
-    )
-    (pin "CS_SD" input (at 101.6 107.95 0)
-      (effects (font (size 1.27 1.27)) (justify right))
-    )
+    (pin "MOSI_FC" input (at 101.6 110.49 0)
+      (effects (font (size 1.27 1.27)) (justify right))
+    )
+    (pin "MISO_FC" output (at 101.6 113.03 0)
+      (effects (font (size 1.27 1.27)) (justify right))
+    )
+    (pin "WP_FC" input (at 101.6 118.11 0)
+      (effects (font (size 1.27 1.27)) (justify right))
+    )
+    (pin "HOLD_FC" input (at 101.6 120.65 0)
+      (effects (font (size 1.27 1.27)) (justify right))
+    )
+    (pin "SCK_FC" input (at 101.6 115.57 0)
+      (effects (font (size 1.27 1.27)) (justify right))
+    )
+    (pin "CS_FC" input (at 101.6 107.95 0)
+      (effects (font (size 1.27 1.27)) (justify right))
+    )

Commit message: Finished routing
Parts:
- added D4, D5: LED, LED_SMD:LED_0402_1005Metric, symbol Device:LED
- added R12, R13: 200, Resistor_SMD:R_0402_1005Metric, symbol Device:R
Connections:
- net +5V: now also R12.1
- net GND: now also D4.1 (K), D5.1 (K)
- net +3.3V renamed +3V3
- net +3V3: now also R13.1
- new net: D5.2 (A), R12.2
- new net: D4.2 (A), R13.2
Other:
- note added: "Power indication LEDs"
Changed lines of the file:
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@@
     (fill (type none))
+  )
+  (rectangle (start 25.4 96.52) (end 49.53 129.54)
+    (stroke (width 0) (type default))
+    (fill (type none))
+  )
+  (text "Power indication LEDs" (at 26.67 100.33 0)
+    (effects (font (size 1.27 1.27) (thickness 0.254) bold) (justify left bottom))
   )
   (text "label these on PCB" (at 25.4 165.1 0)
@@
     )
   )
+  (symbol (lib_id "Device:LED") (at 29.21 118.11 90) (unit 1)
+    (in_bom yes) (on_board yes) (dnp no)
+    (property "Reference" "D5" (at 33.02 119.0625 90)
+      (effects (font (size 1.27 1.27)) (justify right))
+    )
+    (property "Value" "LED" (at 33.02 121.6025 90)
+      (effects (font (size 1.27 1.27)) (justify right))
+    )
+    (property "Footprint" "LED_SMD:LED_0402_1005Metric" (at 29.21 118.11 0)
+      (effects (font (size 1.27 1.27)) hide)
+    )
+    (property "Datasheet" "~" (at 29.21 118.11 0)
+      (effects (font (size 1.27 1.27)) hide)
+    )
+    (pin "1")
+    (pin "2")
+    (instances
+      (project "neptune"
+        (path "/e63e39d7-6ac0-4ffd-8aa3-1841a4541b55/761c8e29-382a-475c-a37a-7201cc9cd0f5"
+          (reference "D5") (unit 1)
+        )
+        (path "/e63e39d7-6ac0-4ffd-8aa3-1841a4541b55"
+          (reference "D4") (unit 1)
+        )
+      )
+    )
+  )
   (symbol (lib_id "Connector:TestPoint") (at 41.91 156.21 0) (unit 1)
     (in_bom yes) (on_board yes) (dnp no)
@@
     )
   )
-  (symbol (lib_id "power:+3.3V") (at 50.8 146.05 0) (unit 1)
+  (symbol (lib_id "power:+3V3") (at 50.8 146.05 0) (unit 1)
     (in_bom yes) (on_board yes) (dnp no) (fields_autoplaced)
     (property "Reference" "#PWR033" (at 50.8 149.86 0)
       (effects (font (size 1.27 1.27)) hide)
     )
-    (property "Value" "+3.3V" (at 50.8 142.24 0)
+    (property "Value" "+3V3" (at 50.8 142.24 0)
       (effects (font (size 1.27 1.27)))
     )
@@
         )
       )
-      (project "keyboard"
-        (path "/fc529d87-72d0-4c92-b352-ddcf4c6f7199/55896886-29a1-46d7-b475-726a72adff13"
-          (reference "#PWR06") (unit 1)
+    )
+  )
+  (symbol (lib_id "Device:R") (at 39.37 110.49 0) (unit 1)
+    (in_bom yes) (on_board yes) (dnp no) (fields_autoplaced)
+    (property "Reference" "R13" (at 41.91 109.855 0)
+      (effects (font (size 1.27 1.27)) (justify left))
+    )
+    (property "Value" "200" (at 41.91 112.395 0)
+      (effects (font (size 1.27 1.27)) (justify left))
+    )
+    (property "Footprint" "Resistor_SMD:R_0402_1005Metric" (at 37.592 110.49 90)
+      (effects (font (size 1.27 1.27)) hide)
+    )
+    (property "Datasheet" "~" (at 39.37 110.49 0)
+      (effects (font (size 1.27 1.27)) hide)
+    )
+    (pin "1")
+    (pin "2")
+    (instances
+      (project "neptune"
+        (path "/e63e39d7-6ac0-4ffd-8aa3-1841a4541b55/761c8e29-382a-475c-a37a-7201cc9cd0f5"
+          (reference "R13") (unit 1)
+        )
+        (path "/e63e39d7-6ac0-4ffd-8aa3-1841a4541b55"
+          (reference "R13") (unit 1)
+        )
+      )
+    )
+  )
+  (symbol (lib_id "power:+3V3") (at 39.37 106.68 0) (unit 1)
+    (in_bom yes) (on_board yes) (dnp no) (fields_autoplaced)
+    (property "Reference" "#PWR04" (at 39.37 110.49 0)
+      (effects (font (size 1.27 1.27)) hide)
+    )
+    (property "Value" "+3V3" (at 39.37 102.87 0)
+      (effects (font (size 1.27 1.27)))
+    )
+    (property "Footprint" "" (at 39.37 106.68 0)
+      (effects (font (size 1.27 1.27)) hide)
+    )
+    (property "Datasheet" "" (at 39.37 106.68 0)
+      (effects (font (size 1.27 1.27)) hide)
+    )
+    (pin "1")
+    (instances
+      (project "neptune"
+        (path "/e63e39d7-6ac0-4ffd-8aa3-1841a4541b55/761c8e29-382a-475c-a37a-7201cc9cd0f5"
+          (reference "#PWR04") (unit 1)
+        )
+        (path "/e63e39d7-6ac0-4ffd-8aa3-1841a4541b55"
+          (reference "#PWR049") (unit 1)
+        )
+      )
+    )
+  )
+  (symbol (lib_id "Device:LED") (at 39.37 118.11 90) (unit 1)
+    (in_bom yes) (on_board yes) (dnp no) (fields_autoplaced)
+    (property "Reference" "D4" (at 43.18 119.0625 90)
+      (effects (font (size 1.27 1.27)) (justify right))
+    )
+    (property "Value" "LED" (at 43.18 121.6025 90)
+      (effects (font (size 1.27 1.27)) (justify right))
+    )
+    (property "Footprint" "LED_SMD:LED_0402_1005Metric" (at 39.37 118.11 0)
+      (effects (font (size 1.27 1.27)) hide)
+    )
+    (property "Datasheet" "~" (at 39.37 118.11 0)
+      (effects (font (size 1.27 1.27)) hide)
+    )
+    (pin "1")
+    (pin "2")
+    (instances
+      (project "neptune"
+        (path "/e63e39d7-6ac0-4ffd-8aa3-1841a4541b55/761c8e29-382a-475c-a37a-7201cc9cd0f5"
+          (reference "D4") (unit 1)
+        )
+        (path "/e63e39d7-6ac0-4ffd-8aa3-1841a4541b55"
+          (reference "D5") (unit 1)
+        )
+      )
+    )
+  )
+  (symbol (lib_name "GND_1") (lib_id "power:GND") (at 39.37 121.92 0) (unit 1)
+    (in_bom yes) (on_board yes) (dnp no) (fields_autoplaced)
+    (property "Reference" "#PWR050" (at 39.37 128.27 0)
+      (effects (font (size 1.27 1.27)) hide)
+    )
+    (property "Value" "GND" (at 39.37 127 0)
+      (effects (font (size 1.27 1.27)))
+    )
+    (property "Footprint" "" (at 39.37 121.92 0)
+      (effects (font (size 1.27 1.27)) hide)
+    )
+    (property "Datasheet" "" (at 39.37 121.92 0)
+      (effects (font (size 1.27 1.27)) hide)
+    )
+    (pin "1")
+    (instances
+      (project "neptune"
+        (path "/e63e39d7-6ac0-4ffd-8aa3-1841a4541b55/761c8e29-382a-475c-a37a-7201cc9cd0f5"
+          (reference "#PWR050") (unit 1)
+        )
+        (path "/e63e39d7-6ac0-4ffd-8aa3-1841a4541b55"
+          (reference "#PWR050") (unit 1)
+        )
+      )
+    )
+  )
+  (symbol (lib_name "+5V_1") (lib_id "power:+5V") (at 29.21 106.68 0) (unit 1)
+    (in_bom yes) (on_board yes) (dnp no) (fields_autoplaced)
+    (property "Reference" "#PWR03" (at 29.21 110.49 0)
+      (effects (font (size 1.27 1.27)) hide)
+    )
+    (property "Value" "+5V" (at 29.21 102.87 0)
+      (effects (font (size 1.27 1.27)))
+    )
+    (property "Footprint" "" (at 29.21 106.68 0)
+      (effects (font (size 1.27 1.27)) hide)
+    )
+    (property "Datasheet" "" (at 29.21 106.68 0)
+      (effects (font (size 1.27 1.27)) hide)
+    )
+    (pin "1")
+    (instances
+      (project "neptune"
+        (path "/e63e39d7-6ac0-4ffd-8aa3-1841a4541b55/761c8e29-382a-475c-a37a-7201cc9cd0f5"
+          (reference "#PWR03") (unit 1)
+        )
+        (path "/e63e39d7-6ac0-4ffd-8aa3-1841a4541b55"
+          (reference "#PWR03") (unit 1)
         )
       )
@@
     )
   )
+  (symbol (lib_id "Device:R") (at 29.21 110.49 0) (unit 1)
+    (in_bom yes) (on_board yes) (dnp no) (fields_autoplaced)
+    (property "Reference" "R12" (at 31.75 109.855 0)
+      (effects (font (size 1.27 1.27)) (justify left))
+    )
+    (property "Value" "200" (at 31.75 112.395 0)
+      (effects (font (size 1.27 1.27)) (justify left))
+    )
+    (property "Footprint" "Resistor_SMD:R_0402_1005Metric" (at 27.432 110.49 90)
+      (effects (font (size 1.27 1.27)) hide)
+    )
+    (property "Datasheet" "~" (at 29.21 110.49 0)
+      (effects (font (size 1.27 1.27)) hide)
+    )
+    (pin "1")
+    (pin "2")
+    (instances
+      (project "neptune"
+        (path "/e63e39d7-6ac0-4ffd-8aa3-1841a4541b55/761c8e29-382a-475c-a37a-7201cc9cd0f5"
+          (reference "R12") (unit 1)
+        )
+        (path "/e63e39d7-6ac0-4ffd-8aa3-1841a4541b55"
+          (reference "R12") (unit 1)
+        )
+      )
+    )
+  )
   (symbol (lib_id "power:VBUS") (at 33.02 146.05 0) (unit 1)
     (in_bom yes) (on_board yes) (dnp no) (fields_autoplaced)
@@
         )
       )
+    )
+  )
+  (symbol (lib_name "GND_1") (lib_id "power:GND") (at 29.21 121.92 0) (unit 1)
+    (in_bom yes) (on_board yes) (dnp no) (fields_autoplaced)
+    (property "Reference" "#PWR049" (at 29.21 128.27 0)
+      (effects (font (size 1.27 1.27)) hide)
+    )
+    (property "Value" "GND" (at 29.21 127 0)
+      (effects (font (size 1.27 1.27)))
+    )
+    (property "Footprint" "" (at 29.21 121.92 0)
+      (effects (font (size 1.27 1.27)) hide)
+    )
+    (property "Datasheet" "" (at 29.21 121.92 0)
+      (effects (font (size 1.27 1.27)) hide)
+    )
+    (pin "1")
+    (instances
+      (project "neptune"
+        (path "/e63e39d7-6ac0-4ffd-8aa3-1841a4541b55/761c8e29-382a-475c-a37a-7201cc9cd0f5"
+          (reference "#PWR049") (unit 1)
+        )
+        (path "/e63e39d7-6ac0-4ffd-8aa3-1841a4541b55"
+          (reference "#PWR04") (unit 1)
+        )
+      )
