File: neptune/power.kicad_sch (KiCad schematic)
At the start: 30 parts, among them Q1 Si2301-TP, Q2 AO3401A, U1 ADR5040ARTZ-2.048, U2 LM393, U3 TPS54331D, U4 LP3993-33B3F

Commit message: Continued routing
Parts:
- C11: footprint Capacitor_SMD:C_0805_2012Metric -> Capacitor_SMD:C_0603_1608Metric
Changed lines of the file:
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@@
       (effects (font (size 1.27 1.27)) (justify left))
     )
-    (property "Footprint" "Capacitor_SMD:C_0805_2012Metric" (at 241.935 45.72 0)
+    (property "Footprint" "Capacitor_SMD:C_0603_1608Metric" (at 241.935 45.72 0)
       (effects (font (size 1.27 1.27)) hide)
     )

Commit message: Routed 3.3V stepdown, added indicator LEDs
Parts:
- added D4, D5: LED, LED_SMD:LED_0402_1005Metric, symbol Device:LED
- added R12, R13: 200, Resistor_SMD:R_0402_1005Metric, symbol Device:R
- C2, C4: footprint Capacitor_SMD:C_0805_2012Metric_Pad1.18x1.45mm_HandSolder -> Capacitor_SMD:C_0603_1608Metric
Connections:
- net +5V: now also R12.1
- net GND: now also D4.1 (K), D5.1 (K)
- net +3.3V renamed +3V3
- net +3V3: now also R13.1
- new net: D4.2 (A), R13.2
- new net: D5.2 (A), R12.2
Other:
- note added: "Power indication LEDs"

Commit message: Finished routing
Parts:
- removed D4, D5: LED, LED_SMD:LED_0402_1005Metric, symbol Device:LED
- removed R12, R13: 200, Resistor_SMD:R_0402_1005Metric, symbol Device:R
Other:
- note removed: "Power indication LEDs"
Changed lines of the file:
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@@
     (stroke (width 0) (type default))
-  )
-  (rectangle (start 232.41 105.41) (end 256.54 138.43)
-    (stroke (width 0) (type default))
-    (fill (type none))
   )
   (text "Circuit protection" (at 15.24 19.05 0)
     (effects (font (size 2.3 2.3) italic) (justify left bottom))
-  )
-  (text "Power indication LEDs" (at 233.68 109.22 0)
-    (effects (font (size 1.27 1.27) (thickness 0.254) bold) (justify left bottom))
   )
   (text "3.3V stepdown" (at 125.73 73.66 0)
@@
     )
   )
-  (symbol (lib_name "GND_1") (lib_id "power:GND") (at 246.38 130.81 0) (unit 1)
-    (in_bom yes) (on_board yes) (dnp no) (fields_autoplaced)
-    (property "Reference" "#PWR050" (at 246.38 137.16 0)
-      (effects (font (size 1.27 1.27)) hide)
-    )
-    (property "Value" "GND" (at 246.38 135.89 0)
-      (effects (font (size 1.27 1.27)))
-    )
-    (property "Footprint" "" (at 246.38 130.81 0)
-      (effects (font (size 1.27 1.27)) hide)
-    )
-    (property "Datasheet" "" (at 246.38 130.81 0)
-      (effects (font (size 1.27 1.27)) hide)
-    )
-    (pin "1")
-    (instances
-      (project "neptune"
-        (path "/e63e39d7-6ac0-4ffd-8aa3-1841a4541b55/761c8e29-382a-475c-a37a-7201cc9cd0f5"
-          (reference "#PWR050") (unit 1)
-        )
-      )
-    )
-  )
   (symbol (lib_id "power:VDC") (at 49.53 83.82 0) (unit 1)
     (in_bom yes) (on_board yes) (dnp no) (fields_autoplaced)
@@
         (path "/fc529d87-72d0-4c92-b352-ddcf4c6f7199/55896886-29a1-46d7-b475-726a72adff13"
           (reference "#PWR09") (unit 1)
-        )
-      )
-    )
-  )
-  (symbol (lib_name "GND_1") (lib_id "power:GND") (at 236.22 130.81 0) (unit 1)
-    (in_bom yes) (on_board yes) (dnp no) (fields_autoplaced)
-    (property "Reference" "#PWR049" (at 236.22 137.16 0)
-      (effects (font (size 1.27 1.27)) hide)
-    )
-    (property "Value" "GND" (at 236.22 135.89 0)
-      (effects (font (size 1.27 1.27)))
-    )
-    (property "Footprint" "" (at 236.22 130.81 0)
-      (effects (font (size 1.27 1.27)) hide)
-    )
-    (property "Datasheet" "" (at 236.22 130.81 0)
-      (effects (font (size 1.27 1.27)) hide)
-    )
-    (pin "1")
-    (instances
-      (project "neptune"
-        (path "/e63e39d7-6ac0-4ffd-8aa3-1841a4541b55/761c8e29-382a-475c-a37a-7201cc9cd0f5"
-          (reference "#PWR049") (unit 1)
         )
       )
@@
     )
   )
-  (symbol (lib_id "Device:LED") (at 246.38 127 90) (unit 1)
-    (in_bom yes) (on_board yes) (dnp no) (fields_autoplaced)
-    (property "Reference" "D4" (at 250.19 127.9525 90)
-      (effects (font (size 1.27 1.27)) (justify right))
-    )
-    (property "Value" "LED" (at 250.19 130.4925 90)
-      (effects (font (size 1.27 1.27)) (justify right))
-    )
-    (property "Footprint" "LED_SMD:LED_0402_1005Metric" (at 246.38 127 0)
-      (effects (font (size 1.27 1.27)) hide)
-    )
-    (property "Datasheet" "~" (at 246.38 127 0)
-      (effects (font (size 1.27 1.27)) hide)
-    )
-    (pin "1")
-    (pin "2")
-    (instances
-      (project "neptune"
-        (path "/e63e39d7-6ac0-4ffd-8aa3-1841a4541b55/761c8e29-382a-475c-a37a-7201cc9cd0f5"
-          (reference "D4") (unit 1)
-        )
-      )
-    )
-  )
   (symbol (lib_id "Device:C_Small") (at 142.875 88.9 0) (unit 1)
     (in_bom yes) (on_board yes) (dnp no)
@@
     )
   )
-  (symbol (lib_id "power:+3V3") (at 246.38 115.57 0) (unit 1)
-    (in_bom yes) (on_board yes) (dnp no) (fields_autoplaced)
-    (property "Reference" "#PWR04" (at 246.38 119.38 0)
-      (effects (font (size 1.27 1.27)) hide)
-    )
-    (property "Value" "+3V3" (at 246.38 111.76 0)
-      (effects (font (size 1.27 1.27)))
-    )
-    (property "Footprint" "" (at 246.38 115.57 0)
-      (effects (font (size 1.27 1.27)) hide)
-    )
-    (property "Datasheet" "" (at 246.38 115.57 0)
-      (effects (font (size 1.27 1.27)) hide)
-    )
-    (pin "1")
-    (instances
-      (project "neptune"
-        (path "/e63e39d7-6ac0-4ffd-8aa3-1841a4541b55/761c8e29-382a-475c-a37a-7201cc9cd0f5"
-          (reference "#PWR04") (unit 1)
-        )
-      )
-    )
-  )
   (symbol (lib_id "Device:R_Small") (at 34.29 46.99 180) (unit 1)
     (in_bom yes) (on_board yes) (dnp no)
@@
         (path "/e63e39d7-6ac0-4ffd-8aa3-1841a4541b55/761c8e29-382a-475c-a37a-7201cc9cd0f5"
           (reference "C1") (unit 1)
-        )
-      )
-    )
-  )
-  (symbol (lib_id "Device:R") (at 246.38 119.38 0) (unit 1)
-    (in_bom yes) (on_board yes) (dnp no) (fields_autoplaced)
-    (property "Reference" "R13" (at 248.92 118.745 0)
-      (effects (font (size 1.27 1.27)) (justify left))
-    )
-    (property "Value" "200" (at 248.92 121.285 0)
-      (effects (font (size 1.27 1.27)) (justify left))
-    )
-    (property "Footprint" "Resistor_SMD:R_0402_1005Metric" (at 244.602 119.38 90)
-      (effects (font (size 1.27 1.27)) hide)
-    )
-    (property "Datasheet" "~" (at 246.38 119.38 0)
-      (effects (font (size 1.27 1.27)) hide)
-    )
-    (pin "1")
-    (pin "2")
-    (instances
-      (project "neptune"
-        (path "/e63e39d7-6ac0-4ffd-8aa3-1841a4541b55/761c8e29-382a-475c-a37a-7201cc9cd0f5"
-          (reference "R13") (unit 1)
         )
       )
@@
     )
   )
-  (symbol (lib_name "+5V_1") (lib_id "power:+5V") (at 236.22 115.57 0) (unit 1)
-    (in_bom yes) (on_board yes) (dnp no) (fields_autoplaced)
-    (property "Reference" "#PWR03" (at 236.22 119.38 0)
-      (effects (font (size 1.27 1.27)) hide)
-    )
-    (property "Value" "+5V" (at 236.22 111.76 0)
-      (effects (font (size 1.27 1.27)))
-    )
-    (property "Footprint" "" (at 236.22 115.57 0)
-      (effects (font (size 1.27 1.27)) hide)
-    )
-    (property "Datasheet" "" (at 236.22 115.57 0)
-      (effects (font (size 1.27 1.27)) hide)
-    )
-    (pin "1")
-    (instances
-      (project "neptune"
-        (path "/e63e39d7-6ac0-4ffd-8aa3-1841a4541b55/761c8e29-382a-475c-a37a-7201cc9cd0f5"
-          (reference "#PWR03") (unit 1)
-        )
-      )
-    )
-  )
   (symbol (lib_id "SRU1048-100Y:SRU1048-100Y") (at 222.885 38.1 0) (unit 1)
     (in_bom yes) (on_board yes) (dnp no) (fields_autoplaced)
@@
         (path "/e63e39d7-6ac0-4ffd-8aa3-1841a4541b55/761c8e29-382a-475c-a37a-7201cc9cd0f5"
           (reference "L1") (unit 1)
-        )
-      )
-    )
-  )
-  (symbol (lib_id "Device:LED") (at 236.22 127 90) (unit 1)
-    (in_bom yes) (on_board yes) (dnp no)
-    (property "Reference" "D5" (at 240.03 127.9525 90)
-      (effects (font (size 1.27 1.27)) (justify right))
-    )
-    (property "Value" "LED" (at 240.03 130.4925 90)
-      (effects (font (size 1.27 1.27)) (justify right))
-    )
-    (property "Footprint" "LED_SMD:LED_0402_1005Metric" (at 236.22 127 0)
-      (effects (font (size 1.27 1.27)) hide)
-    )
-    (property "Datasheet" "~" (at 236.22 127 0)
-      (effects (font (size 1.27 1.27)) hide)
-    )
-    (pin "1")
-    (pin "2")
-    (instances
-      (project "neptune"
-        (path "/e63e39d7-6ac0-4ffd-8aa3-1841a4541b55/761c8e29-382a-475c-a37a-7201cc9cd0f5"
-          (reference "D5") (unit 1)
         )
       )
@@
         )
       )
-    )
-  )
-  (symbol (lib_id "Device:R") (at 236.22 119.38 0) (unit 1)
-    (in_bom yes) (on_board yes) (dnp no) (fields_autoplaced)
-    (property "Reference" "R12" (at 238.76 118.745 0)
-      (effects (font (size 1.27 1.27)) (justify left))
-    )
-    (property "Value" "200" (at 238.76 121.285 0)
-      (effects (font (size 1.27 1.27)) (justify left))
-    )
-    (property "Footprint" "Resistor_SMD:R_0402_1005Metric" (at 234.442 119.38 90)
-      (effects (font (size 1.27 1.27)) hide)
-    )
-    (property "Datasheet" "~" (at 236.22 119.38 0)
-      (effects (font (size 1.27 1.27)) hide)
-    )
-    (pin "1")
-    (pin "2")
-    (instances
-      (project "neptune"
-        (path "/e63e39d7-6ac0-4ffd-8aa3-1841a4541b55/761c8e29-382a-475c-a37a-7201cc9cd0f5"
-          (reference "R12") (unit 1)
-        )
-      )
